File: design/scale_hx711/nRF.sch (KiCad schematic (older format))
At the start: 30 parts, among them J2 Conn_02x03_Odd_Even, Q1 IRLML6401, SW1 SW_SPST, SW2 ON/OFF switch, U1 MDBT42Q, Y1 Q13FC1350000400

Commit message: Adds new footprints, and BoM.
Parts:
- BT1: renamed from BT?; footprint (none) -> Connector_JST:JST_XH_B2B-XH-AM_1x02_P2.50mm_Vertical
- D1: renamed from D?; footprint (none) -> LED_SMD:LED_0603_1608Metric_Castellated
- J1: renamed from J?; footprint (none) -> Footprint_nrf_scale:Micro_usb_connector_4_THT_pads
- Q1: footprint sense_fp:SOT-23 -> Package_TO_SOT_SMD:SOT-23
- R1, R2, R3: renamed from R?; footprint (none) -> Resistor_SMD:R_0603_1608Metric_Pad1.05x0.95mm_HandSolder
- U2: renamed from U?; footprint (none) -> Package_TO_SOT_SMD:SOT-23-6_Handsoldering
- gave numbers to parts that had none: 5
Changed lines of the file:
@@
 F 0 "Q1" V 6800 1600 50  0000 R CNN
 F 1 "IRLML6401" V 7100 1600 50  0000 R CNN
-F 2 "sense_fp:SOT-23" H 7100 1550 29  0001 C CNN
+F 2 "Package_TO_SOT_SMD:SOT-23" H 7100 1550 29  0001 C CNN
 F 3 "" H 6900 1450 60  0000 C CNN
 	1    6900 1450
@@
 	9510 2640 10150 2640
 $Comp
-L sense:Battery_Cell BT?
+L sense:Battery_Cell BT1
 U 1 1 5E71D413
 P 5000 1800
-F 0 "BT?" H 5118 1896 50  0000 L CNN
+F 0 "BT1" H 5118 1896 50  0000 L CNN
 F 1 "Battery_Cell" H 5118 1805 50  0000 L CNN
-F 2 "" V 5000 1860 50  0001 C CNN
+F 2 "Connector_JST:JST_XH_B2B-XH-AM_1x02_P2.50mm_Vertical" V 5000 1860 50  0001 C CNN
 F 3 "" V 5000 1860 50  0001 C CNN
 	1    5000 1800
@@
 $EndComp
 $Comp
-L sense:GND #PWR?
+L sense:GND #PWR0101
 U 1 1 5E5F466B
 P 6900 2150
-F 0 "#PWR?" H 6900 1900 50  0001 C CNN
+F 0 "#PWR0101" H 6900 1900 50  0001 C CNN
 F 1 "GND" H 6900 2000 50  0000 C CNN
 F 2 "" H 6900 2150 60  0000 C CNN
@@
 P 9300 1450
 AR Path="/5E60E4CD" Ref="U?"  Part="1"
-AR Path="/5E602405/5E60E4CD" Ref="U?"  Part="1"
-F 0 "U?" H 9300 1792 50  0000 C CNN
+AR Path="/5E602405/5E60E4CD" Ref="U3"  Part="1"
+F 0 "U3" H 9300 1792 50  0000 C CNN
 F 1 "TPS7A0233PDBV" H 9300 1701 50  0000 C CNN
 F 2 "Package_TO_SOT_SMD:SOT-23-5" H 9300 1775 50  0001 C CIN
@@
 	8650 1350 8500 1350
 $Comp
-L sense:C C?
+L sense:C C8
 U 1 1 5E6167BD
 P 8500 1550
-F 0 "C?" H 8525 1650 50  0000 L CNN
+F 0 "C8" H 8525 1650 50  0000 L CNN
 F 1 "1uF" H 8525 1450 50  0000 L CNN
 F 2 "sense_fp:C_1206_3216Metric" H 8538 1400 30  0001 C CNN
@@
 	8500 1750 8500 1700
 $Comp
-L sense:GND #PWR?
+L sense:GND #PWR0102
 U 1 1 5E6167C4
 P 8500 1750
-F 0 "#PWR?" H 8500 1500 50  0001 C CNN
+F 0 "#PWR0102" H 8500 1500 50  0001 C CNN
 F 1 "GND" H 8500 1600 50  0000 C CNN
 F 2 "" H 8500 1750 60  0000 C CNN
@@
 Connection ~ 8500 1350
 $Comp
-L sense:C C?
+L sense:C C9
 U 1 1 5E6204F3
 P 9800 1550
-F 0 "C?" H 9825 1650 50  0000 L CNN
+F 0 "C9" H 9825 1650 50  0000 L CNN
 F 1 "1uF" H 9825 1450 50  0000 L CNN
 F 2 "sense_fp:C_1206_3216Metric" H 9838 1400 30  0001 C CNN
@@
 	9800 1750 9800 1700
 $Comp
-L sense:GND #PWR?
+L sense:GND #PWR0103
 U 1 1 5E6204FA
 P 9800 1750
-F 0 "#PWR?" H 9800 1500 50  0001 C CNN
+F 0 "#PWR0103" H 9800 1500 50  0001 C CNN
 F 1 "GND" H 9800 1600 50  0000 C CNN
 F 2 "" H 9800 1750 60  0000 C CNN
@@
 $EndComp
 $Comp
-L sense:GND #PWR?
+L sense:GND #PWR0104
 U 1 1 5E6228FD
 P 9300 1800
-F 0 "#PWR?" H 9300 1550 50  0001 C CNN
+F 0 "#PWR0104" H 9300 1550 50  0001 C CNN
 F 1 "GND" H 9300 1650 50  0000 C CNN
 F 2 "" H 9300 1800 60  0000 C CNN
@@
 3.3 V low Iq regulator
 $Comp
-L sense:BQ21040 U?
+L sense:BQ21040 U2
 U 1 1 5E71D41B
 P 3300 1650
-F 0 "U?" H 3300 2115 50  0000 C CNN
+F 0 "U2" H 3300 2115 50  0000 C CNN
 F 1 "BQ21040" H 3300 2024 50  0000 C CNN
-F 2 "" H 3300 1650 50  0001 C CNN
+F 2 "Package_TO_SOT_SMD:SOT-23-6_Handsoldering" H 3300 1650 50  0001 C CNN
 F 3 "http://www.ti.com/lit/ds/symlink/bq21040.pdf" H 3300 1650 50  0001 C CNN
 	1    3300 1650
@@
 $EndComp
 $Comp
-L sense:C C?
+L sense:C C2
 U 1 1 5E71D41C
 P 2150 1800
-F 0 "C?" H 2175 1900 50  0000 L CNN
+F 0 "C2" H 2175 1900 50  0000 L CNN
 F 1 "1uF" H 2000 1700 50  0000 L CNN
 F 2 "sense_fp:C_1206_3216Metric" H 2188 1650 30  0001 C CNN
@@
 	2150 2250 2150 1950
 $Comp
-L sense:GND #PWR?
+L sense:GND #PWR0105
 U 1 1 5E8524E4
 P 2150 2250
-F 0 "#PWR?" H 2150 2000 50  0001 C CNN
+F 0 "#PWR0105" H 2150 2000 50  0001 C CNN
 F 1 "GND" H 2150 2100 50  0000 C CNN
 F 2 "" H 2150 2250 60  0000 C CNN
@@
 	2450 1650 2450 1750
 $Comp
-L sense:R R?
+L sense:R R1
 U 1 1 5E71D41E
 P 2450 1900
-F 0 "R?" H 2350 1900 50  0000 C CNN
+F 0 "R1" H 2350 1900 50  0000 C CNN
 F 1 "1.1k" V 2450 1900 50  0000 C CNN
-F 2 "" V 2380 1900 50  0001 C CNN
+F 2 "Resistor_SMD:R_0603_1608Metric_Pad1.05x0.95mm_HandSolder" V 2380 1900 50  0001 C CNN
 F 3 "" H 2450 1900 50  0001 C CNN
 	1    2450 1900
@@
 $EndComp
 $Comp
-L sense:GND #PWR?
+L sense:GND #PWR0106
 U 1 1 5E71D41F
 P 2450 2250
-F 0 "#PWR?" H 2450 2000 50  0001 C CNN
+F 0 "#PWR0106" H 2450 2000 50  0001 C CNN
 F 1 "GND" H 2450 2100 50  0000 C CNN
 F 2 "" H 2450 2250 60  0000 C CNN
@@
 	2450 2250 2450 2050
 $Comp
-L sense:R R?
+L sense:R R2
 U 1 1 5E71D420
 P 2750 2050
-F 0 "R?" H 2650 2050 50  0000 C CNN
+F 0 "R2" H 2650 2050 50  0000 C CNN
 F 1 "10k" V 2750 2050 50  0000 C CNN
-F 2 "" V 2680 2050 50  0001 C CNN
+F 2 "Resistor_SMD:R_0603_1608Metric_Pad1.05x0.95mm_HandSolder" V 2680 2050 50  0001 C CNN
 F 3 "" H 2750 2050 50  0001 C CNN
 	1    2750 2050
@@
 $EndComp
 $Comp
-L sense:GND #PWR?
+L sense:GND #PWR0107
 U 1 1 5E71D421
 P 2750 2250
-F 0 "#PWR?" H 2750 2000 50  0001 C CNN
+F 0 "#PWR0107" H 2750 2000 50  0001 C CNN
 F 1 "GND" H 2750 2100 50  0000 C CNN
 F 2 "" H 2750 2250 60  0000 C CNN
@@
 	2750 1850 2900 1850
 $Comp
-L sense:R R?
+L sense:R R3
 U 1 1 5E71D422
 P 3950 1650
-F 0 "R?" V 3850 1650 50  0000 C CNN
+F 0 "R3" V 3850 1650 50  0000 C CNN
 F 1 "1.1k" V 3950 1650 50  0000 C CNN
-F 2 "" V 3880 1650 50  0001 C CNN
+F 2 "Resistor_SMD:R_0603_1608Metric_Pad1.05x0.95mm_HandSolder" V 3880 1650 50  0001 C CNN
 F 3 "" H 3950 1650 50  0001 C CNN
 	1    3950 1650
@@
 	3700 1650 3800 1650
 $Comp
-L sense:C C?
+L sense:C C7
 U 1 1 5E8AA9EC
 P 4650 1950
-F 0 "C?" H 4675 2050 50  0000 L CNN
+F 0 "C7" H 4675 2050 50  0000 L CNN
 F 1 "1uF" H 4500 1850 50  0000 L CNN
 F 2 "sense_fp:C_1206_3216Metric" H 4688 1800 30  0001 C CNN
@@
 $EndComp
 $Comp
-L sense:GND #PWR?
+L sense:GND #PWR0108
 U 1 1 5E71D424
 P 4650 2150
-F 0 "#PWR?" H 4650 1900 50  0001 C CNN
+F 0 "#PWR0108" H 4650 1900 50  0001 C CNN
 F 1 "GND" H 4650 2000 50  0000 C CNN
 F 2 "" H 4650 2150 60  0000 C CNN
@@
 	7100 1350 7550 1350
 $Comp
-L sense:LED D?
+L sense:LED D1
 U 1 1 5E71D425
 P 4350 1650
-F 0 "D?" H 4350 1750 50  0000 C CNN
+F 0 "D1" H 4350 1750 50  0000 C CNN
 F 1 "LED" H 4350 1500 50  0000 C CNN
-F 2 "" H 4350 1650 50  0001 C CNN
+F 2 "LED_SMD:LED_0603_1608Metric_Castellated" H 4350 1650 50  0001 C CNN
 F 3 "" H 4350 1650 50  0001 C CNN
 	1    4350 1650
@@
 	4200 1650 4100 1650
 $Comp
-L sense:GND #PWR?
+L sense:GND #PWR0109
 U 1 1 5E94018F
 P 3300 2250
-F 0 "#PWR?" H 3300 2000 50  0001 C CNN
+F 0 "#PWR0109" H 3300 2000 50  0001 C CNN
 F 1 "GND" H 3300 2100 50  0000 C CNN
 F 2 "" H 3300 2250 60  0000 C CNN
@@
 	3300 2250 3300 2150
 $Comp
-L Connector:USB_B_Micro J?
+L Connector:USB_B_Micro J1
 U 1 1 5E9553FD
 P 1050 1650
-F 0 "J?" H 1107 2117 50  0000 C CNN
+F 0 "J1" H 1107 2117 50  0000 C CNN
 F 1 "USB_B_Micro" H 1107 2026 50  0000 C CNN
-F 2 "" H 1200 1600 50  0001 C CNN
+F 2 "Footprint_nrf_scale:Micro_usb_connector_4_THT_pads" H 1200 1600 50  0001 C CNN
 F 3 "~" H 1200 1600 50  0001 C CNN
 	1    1050 1650
@@
 $EndComp
 $Comp
-L sense:GND #PWR?
+L sense:GND #PWR0110
 U 1 1 5E71D428
 P 1050 2150
-F 0 "#PWR?" H 1050 1900 50  0001 C CNN
+F 0 "#PWR0110" H 1050 1900 50  0001 C CNN
 F 1 "GND" H 1050 2000 50  0000 C CNN
 F 2 "" H 1050 2150 60  0000 C CNN
