File: design/scale_hx711/nRF.sch (KiCad schematic (older format))
At the start: 30 parts, among them J1 USB_B_Micro, J2 Conn_02x03_Odd_Even, Q1 IRLML6401, SW1 SW_SPST, SW2 ON/OFF switch, U1 MDBT42Q, U2 BQ21040, U3 TPS7A0233PDBV, Y1 Q13FC1350000400

Commit message: PCB Files added, for scale_hx711
Connections:
- net 10V_LDO_EN: now also U1.20 (P0.07); no longer U1.21 (P0.08)
- net BOOST_EN: now also U1.21 (P0.08); no longer U1.20 (P0.07)
- net GND: now also J2.4 (Pin_4); no longer J2.6 (Pin_6)
- net HX711_CLK: now also U1.27 (P0.13); no longer U1.25 (P0.11)
- net HX711_DATA: now also U1.26 (P0.12); no longer U1.27 (P0.13)
- net HX711_RATE: now also U1.25 (P0.11); no longer U1.26 (P0.12)
- net RX: now also J2.5 (Pin_5); no longer J2.2 (Pin_2)
- net TX: now also J2.6 (Pin_6); no longer J2.5 (Pin_5)
- net VDD: now also J2.2 (Pin_2); no longer J2.4 (Pin_4)
- net EINK_BUSY: now reaches U1.2 (P0.25)
- net EINK_RST: now reaches U1.3 (P0.26)
- net EINK_CS: now reaches U1.4 (P0.27)
- net EINK_SCLK: now reaches U1.5 (P0.28/AIN4)
- net EINK_SDIO: now reaches U1.6 (P0.29/AIN5)
- no-connect marks 9 -> 21
Other:
- moved on the sheet: J2
Changed lines of the file:
@@
 Text Label 2550 4580 3    60   ~ 0
 LFCLK_XL2
-Text Label 1350 6975 0    50   ~ 0
+Text Label 1450 6975 0    50   ~ 0
 SWDIO
-Text Label 1350 7075 0    50   ~ 0
+Text Label 1450 7075 0    50   ~ 0
 SWDCLK
-Text Label 2550 6975 2    50   ~ 0
+Text Label 1450 7175 0    50   ~ 0
 RX
-Text Label 1350 7175 0    50   ~ 0
+Text Label 2650 7175 2    50   ~ 0
 TX
 $Comp
 L sense:VDD #PWR05
 U 1 1 5E71D407
-P 2700 7025
-F 0 "#PWR05" H 2700 6875 50  0001 C CNN
-F 1 "VDD" H 2700 7175 50  0000 C CNN
-F 2 "" H 2700 7025 60  0000 C CNN
-F 3 "" H 2700 7025 60  0000 C CNN
-	1    2700 7025
+P 2801 6900
+F 0 "#PWR05" H 2801 6750 50  0001 C CNN
+F 1 "VDD" H 2801 7050 50  0000 C CNN
+F 2 "" H 2801 6900 60  0000 C CNN
+F 3 "" H 2801 6900 60  0000 C CNN
+	1    2801 6900
 	1    0    0    -1
 $EndComp
@@
 Text Notes 1180 3310 0    60   ~ 0
 To use the Internal DC/DC\nregulator we need external\ninductors
-Text Notes 1600 6675 0    60   ~ 0
+Text Notes 1600 6700 0    60   ~ 0
 For programming \nand debugging \nthe nRF controller
 Text Notes 1900 4830 0    60   ~ 0
@@
 L sense:GND #PWR04
 U 1 1 5E71D403
-P 2700 7225
-F 0 "#PWR04" H 2700 6975 50  0001 C CNN
-F 1 "GND" H 2700 7075 50  0000 C CNN
-F 2 "" H 2700 7225 60  0000 C CNN
-F 3 "" H 2700 7225 60  0000 C CNN
-	1    2700 7225
+P 2800 7250
+F 0 "#PWR04" H 2800 7000 50  0001 C CNN
+F 1 "GND" H 2800 7100 50  0000 C CNN
+F 2 "" H 2800 7250 60  0000 C CNN
+F 3 "" H 2800 7250 60  0000 C CNN
+	1    2800 7250
 	1    0    0    -1
 $EndComp
@@
 L sense:Conn_02x03_Odd_Even J2
 U 1 1 5D8500C4
-P 1900 7075
-F 0 "J2" H 1950 7392 50  0000 C CNN
-F 1 "Conn_02x03_Odd_Even" H 1950 7301 50  0000 C CNN
-F 2 "Connector_PinHeader_2.00mm:PinHeader_2x03_P2.00mm_Vertical" H 1900 7075 50  0001 C CNN
-F 3 "~" H 1900 7075 50  0001 C CNN
-	1    1900 7075
-	1    0    0    -1
-$EndComp
-Wire Wire Line
-	2700 7225 2700 7175
-Wire Wire Line
-	2700 7175 2200 7175
-Wire Wire Line
-	2200 7075 2700 7075
-Wire Wire Line
-	2700 7075 2700 7025
-Wire Wire Line
-	2200 6975 2550 6975
-Wire Wire Line
-	1350 6975 1700 6975
-Wire Wire Line
-	1700 7075 1350 7075
-Wire Wire Line
-	1350 7175 1700 7175
+P 2000 7075
+F 0 "J2" H 2050 7392 50  0000 C CNN
+F 1 "Conn_02x03_Odd_Even" H 2050 7301 50  0000 C CNN
+F 2 "Connector_PinHeader_2.00mm:PinHeader_2x03_P2.00mm_Vertical" H 2000 7075 50  0001 C CNN
+F 3 "~" H 2000 7075 50  0001 C CNN
+	1    2000 7075
+	1    0    0    -1
+$EndComp
+Wire Wire Line
+	2300 7175 2650 7175
+Wire Wire Line
+	1450 6975 1800 6975
+Wire Wire Line
+	1800 7075 1450 7075
+Wire Wire Line
+	1450 7175 1800 7175
 $Comp
 L sense:SW_SPST SW1
@@
 NoConn ~ 7220 3400
 NoConn ~ 7220 3500
-$Comp
-L sense:MDBT42Q U1
-U 1 1 5E71D3F5
-P 6020 4100
-F 0 "U1" H 5105 2700 60  0000 C CNN
-F 1 "MDBT42Q" H 6020 4850 60  0000 C CNN
-F 2 "sense_fp:mdbt42Q" H 5820 5200 60  0001 C CNN
-F 3 "" H 5820 5200 60  0000 C CNN
-	1    6020 4100
-	1    0    0    -1
-$EndComp
 Wire Wire Line
 	5520 5650 5520 6300
@@
 Wire Wire Line
 	4820 4800 4200 4800
-Wire Wire Line
-	4820 4700 4200 4700
 Wire Wire Line
 	3965 3450 4820 3450
@@
 Text HLabel 7550 1350 2    50   Output ~ 0
 VBAT
-Text HLabel 7800 4700 2    50   Input ~ 0
+Text HLabel 7800 4800 2    50   Input ~ 0
 HX711_DATA
-Text HLabel 7800 4800 2    50   Output ~ 0
+Text HLabel 7800 4900 2    50   Output ~ 0
 HX711_RATE
-Text HLabel 7800 4900 2    50   BiDi ~ 0
+Text HLabel 7800 4700 2    50   BiDi ~ 0
 HX711_CLK
 Text Label 6120 6300 1    50   ~ 0
 BUTTON
+Text HLabel 6320 6300 3    50   Output ~ 0
+BOOST_EN
 Text HLabel 6220 6300 3    50   Output ~ 0
-BOOST_EN
-Text HLabel 6320 6300 3    50   Output ~ 0
 10V_LDO_EN
 Text HLabel 6020 6300 3    50   Input ~ 0
@@
 NoConn ~ 6520 5650
 Wire Wire Line
-	6220 6300 6220 5650
+	7800 4900 7220 4900
+Wire Wire Line
+	7220 4800 7800 4800
+Wire Wire Line
+	7800 4700 7220 4700
+Text HLabel 4240 4400 0    50   Output ~ 0
+EINK_SDIO
+Text HLabel 4230 4300 0    50   Output ~ 0
+EINK_SCLK
+Text HLabel 4240 4200 0    50   Output ~ 0
+EINK_CS
+Text HLabel 4240 4100 0    50   Output ~ 0
+EINK_RST
+Text HLabel 4240 4000 0    50   Input ~ 0
+EINK_BUSY
+Wire Wire Line
+	4240 4000 4820 4000
+Wire Wire Line
+	4820 4200 4240 4200
+Wire Wire Line
+	4820 4400 4240 4400
+Wire Wire Line
+	2801 6900 2801 6975
+Wire Wire Line
+	2801 6975 2300 6975
+Wire Wire Line
+	2800 7250 2800 7075
+Wire Wire Line
+	2800 7075 2300 7075
+NoConn ~ 4820 4600
+NoConn ~ 4820 4500
+Wire Wire Line
+	4820 4100 4240 4100
+Wire Wire Line
+	4230 4300 4820 4300
+$Comp
+L sense:MDBT42Q U1
+U 1 1 5E71D3F5
+P 6020 4100
+F 0 "U1" H 5105 2700 60  0000 C CNN
+F 1 "MDBT42Q" H 6020 4850 60  0000 C CNN
+F 2 "sense_fp:mdbt42Q" H 5820 5200 60  0001 C CNN
+F 3 "" H 5820 5200 60  0000 C CNN
+	1    6020 4100
+	1    0    0    -1
+$EndComp
+Wire Wire Line
+	4820 4700 4200 4700
+NoConn ~ 5720 5650
+NoConn ~ 5820 5650
+NoConn ~ 5920 5650
+Wire Wire Line
+	6220 5650 6220 6300
 Wire Wire Line
 	6320 5650 6320 6300
-Wire Wire Line
-	7800 4900 7220 4900
-Wire Wire Line
-	7220 4800 7800 4800
-Wire Wire Line
-	7800 4700 7220 4700
+NoConn ~ 7220 4600
+NoConn ~ 7220 4500
+NoConn ~ 7220 4400
+NoConn ~ 7220 4300
+NoConn ~ 7220 4200
+NoConn ~ 7220 4100
+NoConn ~ 7220 3600
 $EndSCHEMATC

Commit message: Adds extra GPIO pins for nrf in scale_hx711
Parts:
- added J4: Conn_01x04, Connector_PinHeader_2.00mm:PinHeader_1x04_P2.00mm_Vertical, symbol Connector_Generic:Conn_01x04
Connections:
- net GPIO3: now reaches U1.28 (TRACE_DATA3/P0.14)
- net GPIO3: now also J4.4 (Pin_4)
- net GPIO2: now reaches U1.29 (TRACE_DATA2/P0.15)
- net GPIO2: now also J4.3 (Pin_3)
- net GPIO1: now reaches U1.30 (TRACE_DATA1/P0.16)
- net GPIO1: now also J4.2 (Pin_2)
- net GPIO0: now reaches U1.31 (P0.17)
- net GPIO0: now also J4.1 (Pin_1)
- no-connect marks 21 -> 17
Changed lines of the file:
@@
 Wire Wire Line
 	6320 5650 6320 6300
-NoConn ~ 7220 4600
-NoConn ~ 7220 4500
-NoConn ~ 7220 4400
-NoConn ~ 7220 4300
 NoConn ~ 7220 4200
 NoConn ~ 7220 4100
 NoConn ~ 7220 3600
+$Comp
+L Connector_Generic:Conn_01x04 J4
+U 1 1 5E6691E5
+P 10400 4450
+F 0 "J4" H 10480 4442 50  0000 L CNN
+F 1 "Conn_01x04" H 10480 4351 50  0000 L CNN
+F 2 "Connector_PinHeader_2.00mm:PinHeader_1x04_P2.00mm_Vertical" H 10400 4450 50  0001 C CNN
+F 3 "~" H 10400 4450 50  0001 C CNN
+	1    10400 4450
+	1    0    0    -1
+$EndComp
+Text Label 9900 4350 0    50   ~ 0
+GPIO0
+Text Label 9900 4450 0    50   ~ 0
+GPIO1
+Text Label 9900 4550 0    50   ~ 0
+GPIO2
+Text Label 9900 4650 0    50   ~ 0
+GPIO3
+Wire Wire Line
+	9900 4650 10200 4650
+Wire Wire Line
+	10200 4550 9900 4550
+Wire Wire Line
+	9900 4450 10200 4450
+Wire Wire Line
+	10200 4350 9900 4350
+Text Label 7800 4300 2    50   ~ 0
+GPIO0
+Text Label 7800 4400 2    50   ~ 0
+GPIO1
+Text Label 7800 4500 2    50   ~ 0
+GPIO2
+Text Label 7800 4600 2    50   ~ 0
+GPIO3
+Wire Wire Line
+	7220 4600 7800 4600
+Wire Wire Line
+	7800 4300 7220 4300
+Wire Wire Line
+	7220 4400 7800 4400
+Wire Wire Line
+	7800 4500 7220 4500
 $EndSCHEMATC

Commit message: BOMs, schematics updated, scale_ltc6915 PCB Design complete.
Parts:
- added Q4: AO3400, Package_TO_SOT_SMD:SOT-23, symbol sense:Q_NMOS_GSD
- added R14, R15: 10k, Resistor_SMD:R_0603_1608Metric_Pad1.05x0.95mm_HandSolder, symbol sense:R
Connections:
- net 10V_LDO_EN: now also U1.21 (P0.08); no longer U1.20 (P0.07)
- net BOOST_EN: now also U1.22 (P0.09/NFC1); no longer U1.21 (P0.08)
- net BUTTON: now also U1.20 (P0.07); no longer U1.19 (P0.06)
- net GND: now also Q4.2 (S)
- net VBAT: now also R14.2
- net Vlc: now also U1.17 (P0.04/AIN2); no longer U1.18 (P0.05/AIN3)
- net BT_LV_EN: now reaches U1.23 (P0.10/NFC2)
- net BT_LV_EN: now also Q4.1 (G)
- new net: Q4.3 (D), R15.1
- new net BT_LV: R14.1, R15.2, U1.18 (P0.05/AIN3)
- no-connect marks 17 -> 15
Other:
- moved on the sheet: C16, J4, SW1
Changed lines of the file:
@@
 L sense:GND #PWR01
 U 1 1 5A8704B4
-P 8770 3120
-F 0 "#PWR01" H 8770 2870 50  0001 C CNN
-F 1 "GND" H 8770 2970 50  0000 C CNN
-F 2 "" H 8770 3120 60  0000 C CNN
-F 3 "" H 8770 3120 60  0000 C CNN
-	1    8770 3120
+P 9060 5740
+F 0 "#PWR01" H 9060 5490 50  0001 C CNN
+F 1 "GND" H 9060 5590 50  0000 C CNN
+F 2 "" H 9060 5740 60  0000 C CNN
+F 3 "" H 9060 5740 60  0000 C CNN
+	1    9060 5740
 	1    0    0    -1
 $EndComp
@@
 Text Notes 6450 1100 0    60   ~ 0
 Reverse polarity protection
-Text Notes 8760 2445 0    60   ~ 0
+Text Notes 9050 5065 0    60   ~ 0
 Button for Tare
 Text Notes 1180 3310 0    60   ~ 0
@@
 L sense:C C16
 U 1 1 5D422270
-P 9510 2900
-F 0 "C16" H 9360 2995 50  0000 L CNN
-F 1 "0.1nF" H 9265 2820 50  0000 L CNN
-F 2 "sense_fp:C_0402_1005Metric" H 9548 2750 30  0001 C CNN
-F 3 "" H 9510 2900 60  0000 C CNN
-	1    9510 2900
+P 9800 5520
+F 0 "C16" H 9650 5615 50  0000 L CNN
+F 1 "0.1nF" H 9555 5440 50  0000 L CNN
+F 2 "sense_fp:C_0402_1005Metric" H 9838 5370 30  0001 C CNN
+F 3 "" H 9800 5520 60  0000 C CNN
+	1    9800 5520
 	-1   0    0    1
 $EndComp
@@
 L sense:GND #PWR032
 U 1 1 5D42FC1A
-P 9510 3110
-F 0 "#PWR032" H 9510 2860 50  0001 C CNN
-F 1 "GND" H 9510 2960 50  0000 C CNN
-F 2 "" H 9510 3110 60  0000 C CNN
-F 3 "" H 9510 3110 60  0000 C CNN
-	1    9510 3110
+P 9800 5730
+F 0 "#PWR032" H 9800 5480 50  0001 C CNN
+F 1 "GND" H 9800 5580 50  0000 C CNN
+F 2 "" H 9800 5730 60  0000 C CNN
+F 3 "" H 9800 5730 60  0000 C CNN
+	1    9800 5730
 	1    0    0    -1
 $EndComp
@@
 L sense:SW_SPST SW1
 U 1 1 5E71D3F6
-P 9160 2640
-F 0 "SW1" H 9160 2765 50  0000 C CNN
-F 1 "SW_SPST" H 9160 2540 50  0000 C CNN
-F 2 "Footprint_nrf_scale:SMD Tactile Switch_3x6x2.5mm" H 9160 2640 50  0001 C CNN
-F 3 "" H 9160 2640 50  0001 C CNN
-	1    9160 2640
+P 9450 5260
+F 0 "SW1" H 9450 5385 50  0000 C CNN
+F 1 "SW_SPST" H 9450 5160 50  0000 C CNN
+F 2 "Footprint_nrf_scale:SMD Tactile Switch_3x6x2.5mm" H 9450 5260 50  0001 C CNN
+F 3 "" H 9450 5260 50  0001 C CNN
+	1    9450 5260
 	1    0    0    -1
 $EndComp
@@
 Wire Wire Line
 	7220 4000 7800 4000
-Text Label 10150 2640 2    50   ~ 0
+Text Label 10440 5260 2    50   ~ 0
 BUTTON
 Wire Wire Line
-	9510 3050 9510 3110
-Wire Wire Line
-	8770 3120 8770 2640
-Wire Wire Line
-	8770 2640 8960 2640
-Wire Wire Line
-	9360 2640 9510 2640
-Wire Wire Line
-	9510 2750 9510 2640
-Connection ~ 9510 2640
-Wire Wire Line
-	9510 2640 10150 2640
+	9800 5670 9800 5730
+Wire Wire Line
+	9060 5740 9060 5260
+Wire Wire Line
+	9060 5260 9250 5260
+Wire Wire Line
+	9650 5260 9800 5260
+Wire Wire Line
+	9800 5370 9800 5260
+Connection ~ 9800 5260
+Wire Wire Line
+	9800 5260 10440 5260
 $Comp
 L sense:Battery_Cell BT1
@@
 Text HLabel 7800 4700 2    50   BiDi ~ 0
 HX711_CLK
-Text Label 6120 6300 1    50   ~ 0
+Text Label 6220 6300 1    50   ~ 0
 BUTTON
+Text HLabel 6420 6300 3    50   Output ~ 0
+BOOST_EN
 Text HLabel 6320 6300 3    50   Output ~ 0
-BOOST_EN
-Text HLabel 6220 6300 3    50   Output ~ 0
 10V_LDO_EN
-Text HLabel 6020 6300 3    50   Input ~ 0
+Text HLabel 5920 6300 3    50   Input ~ 0
 Vlc
 Wire Wire Line
 	6020 6300 6020 5650
 Wire Wire Line
-	6120 5650 6120 6300
-NoConn ~ 6420 5650
-NoConn ~ 6520 5650
+	6320 5650 6320 6300
 Wire Wire Line
 	7800 4900 7220 4900
@@
 NoConn ~ 5720 5650
 NoConn ~ 5820 5650
-NoConn ~ 5920 5650
-Wire Wire Line
-	6220 5650 6220 6300
-Wire Wire Line
-	6320 5650 6320 6300
+Wire Wire Line
+	6420 5650 6420 6300
+Wire Wire Line
+	6520 5650 6520 6300
 NoConn ~ 7220 4200
 NoConn ~ 7220 4100
@@
 L Connector_Generic:Conn_01x04 J4
 U 1 1 5E6691E5
-P 10400 4450
-F 0 "J4" H 10480 4442 50  0000 L CNN
-F 1 "Conn_01x04" H 10480 4351 50  0000 L CNN
-F 2 "Connector_PinHeader_2.00mm:PinHeader_1x04_P2.00mm_Vertical" H 10400 4450 50  0001 C CNN
-F 3 "~" H 10400 4450 50  0001 C CNN
-	1    10400 4450
-	1    0    0    -1
-$EndComp
-Text Label 9900 4350 0    50   ~ 0
+P 10550 4370
+F 0 "J4" H 10630 4362 50  0000 L CNN
+F 1 "Conn_01x04" H 10630 4271 50  0000 L CNN
+F 2 "Connector_PinHeader_2.00mm:PinHeader_1x04_P2.00mm_Vertical" H 10550 4370 50  0001 C CNN
+F 3 "~" H 10550 4370 50  0001 C CNN
+	1    10550 4370
+	1    0    0    -1
+$EndComp
+Text Label 10050 4270 0    50   ~ 0
 GPIO0
-Text Label 9900 4450 0    50   ~ 0
+Text Label 10050 4370 0    50   ~ 0
 GPIO1
-Text Label 9900 4550 0    50   ~ 0
+Text Label 10050 4470 0    50   ~ 0
 GPIO2
-Text Label 9900 4650 0    50   ~ 0
+Text Label 10050 4570 0    50   ~ 0
 GPIO3
 Wire Wire Line
-	9900 4650 10200 4650
-Wire Wire Line
-	10200 4550 9900 4550
-Wire Wire Line
-	9900 4450 10200 4450
-Wire Wire Line
-	10200 4350 9900 4350
+	10050 4570 10350 4570
+Wire Wire Line
+	10350 4470 10050 4470
+Wire Wire Line
+	10050 4370 10350 4370
+Wire Wire Line
+	10350 4270 10050 4270
 Text Label 7800 4300 2    50   ~ 0
 GPIO0
@@
 Wire Wire Line
 	7800 4500 7220 4500
+$Comp
+L sense:Q_NMOS_GSD Q?
+U 1 1 5E7CDED4
+P 10300 3500
+AR Path="/5E60241F/5E7CDED4" Ref="Q?"  Part="1"
+AR Path="/5E602405/5E7CDED4" Ref="Q4"  Part="1"
+F 0 "Q4" H 10506 3546 50  0000 L CNN
+F 1 "AO3400" H 10506 3455 50  0000 L CNN
+F 2 "Package_TO_SOT_SMD:SOT-23" H 10500 3600 50  0001 C CNN
+F 3 "" H 10300 3500 50  0001 C CNN
+	1    10300 3500
+	1    0    0    -1
+$EndComp
+$Comp
+L sense:R R14
+U 1 1 5E7D4334
+P 10400 2560
+F 0 "R14" V 10300 2560 50  0000 C CNN
+F 1 "10k" V 10400 2560 50  0000 C CNN
+F 2 "Resistor_SMD:R_0603_1608Metric_Pad1.05x0.95mm_HandSolder" V 10330 2560 50  0001 C CNN
+F 3 "" H 10400 2560 50  0001 C CNN
+	1    10400 2560
+	-1   0    0    1
+$EndComp
+$Comp
+L sense:R R15
+U 1 1 5E7D8EAA
+P 10400 3050
+F 0 "R15" V 10300 3050 50  0000 C CNN
+F 1 "10k" V 10400 3050 50  0000 C CNN
+F 2 "Resistor_SMD:R_0603_1608Metric_Pad1.05x0.95mm_HandSolder" V 10330 3050 50  0001 C CNN
+F 3 "" H 10400 3050 50  0001 C CNN
+	1    10400 3050
+	-1   0    0    1
+$EndComp
+$Comp
+L sense:GND #PWR0149
+U 1 1 5E7DBBE8
+P 10400 3800
+F 0 "#PWR0149" H 10400 3550 50  0001 C CNN
+F 1 "GND" H 10400 3650 50  0000 C CNN
+F 2 "" H 10400 3800 60  0000 C CNN
+F 3 "" H 10400 3800 60  0000 C CNN
+	1    10400 3800
+	1    0    0    -1
+$EndComp
+Wire Wire Line
+	10400 3800 10400 3700
+Wire Wire Line
+	10400 3200 10400 3300
+Text Label 10400 2200 2    50   ~ 0
+VBAT
+Wire Wire Line
+	10400 2200 10400 2410
+Text Label 9600 3500 0    50   ~ 0
+BT_LV_EN
+Wire Wire Line
+	9600 3500 10100 3500
+Text Label 9600 2800 0    50   ~ 0
+BT_LV
+Wire Wire Line
+	9600 2800 10400 2800
+Wire Wire Line
+	10400 2710 10400 2800
+Connection ~ 10400 2800
+Wire Wire Line
+	10400 2800 10400 2900
+Text Label 6520 6300 1    50   ~ 0
+BT_LV_EN
+Text Label 6020 6300 1    50   ~ 0
+BT_LV
+Wire Wire Line
+	5920 6300 5920 5650
+Wire Wire Line
+	6220 6300 6220 5650
+NoConn ~ 6120 5650
 $EndSCHEMATC

Commit message: DC, CS pins separated, issue fixed. In both scale_hx711 and scale_ltc6915.
Connections:
- net EINK_CS: now also U1.5 (P0.28/AIN4); no longer U1.4 (P0.27)
- net EINK_SCLK: now also U1.6 (P0.29/AIN5); no longer U1.5 (P0.28/AIN4)
- net EINK_SDIO: now also U1.7 (P0.30/AIN6); no longer U1.6 (P0.29/AIN5)
- new net EINK_DC: U1.4 (P0.27)
- no-connect marks 15 -> 14
Changed lines of the file:
@@
 Wire Wire Line
 	7800 4700 7220 4700
-Text HLabel 4240 4400 0    50   Output ~ 0
+Text HLabel 4240 4500 0    50   Output ~ 0
 EINK_SDIO
-Text HLabel 4230 4300 0    50   Output ~ 0
+Text HLabel 4230 4400 0    50   Output ~ 0
 EINK_SCLK
-Text HLabel 4240 4200 0    50   Output ~ 0
+Text HLabel 4240 4300 0    50   Output ~ 0
 EINK_CS
 Text HLabel 4240 4100 0    50   Output ~ 0
@@
 	4240 4000 4820 4000
 Wire Wire Line
-	4820 4200 4240 4200
+	4820 4300 4240 4300
 Wire Wire Line
-	4820 4400 4240 4400
+	4820 4500 4240 4500
 Wire Wire Line
 	2801 6900 2801 6975
@@
 	2800 7075 2300 7075
 NoConn ~ 4820 4600
-NoConn ~ 4820 4500
 Wire Wire Line
 	4820 4100 4240 4100
 Wire Wire Line
-	4230 4300 4820 4300
+	4230 4400 4820 4400
 $Comp
 L sense:MDBT42Q U1
@@
 	6220 6300 6220 5650
 NoConn ~ 6120 5650
+Text HLabel 4240 4200 0    50   Output ~ 0
+EINK_DC
+Wire Wire Line
+	4240 4200 4820 4200
 $EndSCHEMATC
