File: design/scale_hx711/epaper.sch (KiCad schematic (older format))
At the start: 19 parts

Commit message: Adds new footprints, and BoM.
Parts:
- C10, C11, C12, C13, C14, C15, C17, C18, C19, C20, C21: renamed from C?; footprint (none) -> Capacitor_SMD:C_0603_1608Metric_Pad1.05x0.95mm_HandSolder
- D2, D3, D4: renamed from D?; footprint (none) -> Diode_SMD:D_SOD-323_HandSoldering
- EINK1: renamed from EINK?; footprint (none) -> Connector_FFC-FPC:Hirose_FH12-24S-0.5SH_1x24-1MP_P0.50mm_Horizontal
- L3: renamed from L?; footprint (none) -> Footprint_nrf_scale:L_3.5x3.0mm_CD30D22
- Q2: renamed from Q?; footprint (none) -> Package_TO_SOT_SMD:SOT-23
- R4, R5: renamed from R?; footprint (none) -> Resistor_SMD:R_0603_1608Metric_Pad1.05x0.95mm_HandSolder

Commit message: BOMs, schematics updated, scale_ltc6915 PCB Design complete.
Parts:
- R5: footprint Resistor_SMD:R_0603_1608Metric_Pad1.05x0.95mm_HandSolder -> Resistor_SMD:R_1206_3216Metric
Changed lines of the file:
@@
 F 0 "R5" H 2170 4496 50  0000 L CNN
 F 1 "0.47" H 2170 4405 50  0000 L CNN
-F 2 "Resistor_SMD:R_0603_1608Metric_Pad1.05x0.95mm_HandSolder" V 2030 4450 50  0001 C CNN
+F 2 "Resistor_SMD:R_1206_3216Metric" V 2030 4450 50  0001 C CNN
 F 3 "" H 2100 4450 50  0001 C CNN
 	1    2100 4450

Commit message: DC, CS pins separated, issue fixed. In both scale_hx711 and scale_ltc6915.
Connections:
- net EINK_CS: no longer EINK1.11 (D/C#)
- new net EINK_DC: EINK1.11 (D/C#)
Changed lines of the file:
@@
 EINK_CS
 Text HLabel 8500 3000 0    50   Input ~ 0
-EINK_CS
+EINK_DC
 Text HLabel 8500 2900 0    50   Input ~ 0
 EINK_RST
