File: design/scale_ltc6915/epaper.sch (KiCad schematic (older format))
At the start: 19 parts, among them Q2 AO3400

Commit message: DC, CS pins separated, issue fixed. In both scale_hx711 and scale_ltc6915.
Connections:
- net EINK_CS: no longer EINK1.11 (D/C#)
- new net EINK_DS: EINK1.11 (D/C#)
Changed lines of the file:
@@
 EINK_CS
 Text HLabel 8500 3000 0    50   Input ~ 0
-EINK_CS
+EINK_DS
 Text HLabel 8500 2900 0    50   Input ~ 0
 EINK_RST
